Commit message: feat: 同步 Gazebo 仿真进展（地形模型、扩散策略与部署验证）
- lunar_gazebo: 新增 lunar_terrain 地形模型（model.sdf/config + OBJ 网格与贴图），
  lunar_field.world 改为引用真实月面地形
- lunar_env: env.py 大幅扩展；新增 eval_deploy、run_policy_diffusion、
  run_policy_hybrid、record_episode、camera_recorder、var_policy
- lunar_rl: 新增 terrain.py 地形模块、diffusion_actor、train_diffusion_bc、
  collect_surrogate_data、eval_purpose、train_gazebo_bc_vars；
  rewards / rule_policy / surrogate / obs / networks 同步更新
- lunar_control / lunar_descriptions / lunar_task / lunar_bringup:
  控制器参数、URDF、场景配置与资源管理状态机同步
- docs: 新增 gazebo仿真方案、9.27-Gazebo部署验证、9.23-9.28、9.29-10.6、
  目的性与地形感知改造、模型训练方案：目的性增强
- results: 新增仿真演示视频与曲线（模型权重 *.pt 仍排除）
- .gitignore: 排除第三方商业 3D 模型素材 map_model/

File: src/lunar_descriptions/urdf/excavator.urdf.xacro (robot description, xacro)
@@ -1,4 +1,6 @@
 <?xml version="1.0"?>
-<robot xmlns:xacro="http://www.ros.org/wiki/xacro" name="excavator">
+<robot xmlns:xacro="http://www.ros.org/wiki/xacro" name="$(arg name)">
+  <xacro:arg name="name" default="excavator"/>
+  <xacro:arg name="ns" default="excavator"/>
   <xacro:include filename="$(find lunar_descriptions)/urdf/common.xacro"/>
   <!-- ===== 底盘 ===== -->
@@ -90,8 +92,8 @@
     <plugin filename="libgazebo_ros2_control.so" name="gazebo_ros2_control">
       <robot_param>robot_description</robot_param>
-      <robot_param_node>excavator_rsp</robot_param_node>
+      <robot_param_node>$(arg name)_rsp</robot_param_node>
       <parameters>$(find lunar_control)/config/excavator_controllers.yaml</parameters>
       <ros>
-        <namespace>excavator</namespace>
+        <namespace>$(arg ns)</namespace>
       </ros>
     </plugin>

File: src/lunar_descriptions/urdf/hauler.urdf.xacro (robot description, xacro)
@@ -1,4 +1,6 @@
 <?xml version="1.0"?>
-<robot xmlns:xacro="http://www.ros.org/wiki/xacro" name="hauler">
+<robot xmlns:xacro="http://www.ros.org/wiki/xacro" name="$(arg name)">
+  <xacro:arg name="name" default="hauler"/>
+  <xacro:arg name="ns" default="hauler"/>
   <xacro:include filename="$(find lunar_descriptions)/urdf/common.xacro"/>
   <!-- ===== 底盘 ===== -->
@@ -13,4 +15,13 @@
     <xacro:box_inertial mass="9.0" lx="0.46" ly="0.34" lz="0.12"/>
   </link>
+  <!-- 低配重：把重心压到接近地面，抑制料斗倾倒/急停时的倾倒失稳 -->
+  <link name="ballast_link">
+    <xacro:box_inertial mass="4.0" lx="0.34" ly="0.30" lz="0.04"/>
+  </link>
+  <joint name="ballast_joint" type="fixed">
+    <parent link="base_link"/>
+    <child link="ballast_link"/>
+    <origin xyz="0 0 -0.06" rpy="0 0 0"/>
+  </joint>
   <xacro:drive_wheel prefix="left" parent="base_link" xyz="0 0.19 -0.04" rpy="1.5708 0 0" mass="0.5" radius="0.08" width="0.04"/>
   <xacro:drive_wheel prefix="right" parent="base_link" xyz="0 -0.19 -0.04" rpy="1.5708 0 0" mass="0.5" radius="0.08" width="0.04"/>
@@ -39,8 +50,8 @@
     <plugin filename="libgazebo_ros2_control.so" name="gazebo_ros2_control">
       <robot_param>robot_description</robot_param>
-      <robot_param_node>hauler_rsp</robot_param_node>
+      <robot_param_node>$(arg name)_rsp</robot_param_node>
       <parameters>$(find lunar_control)/config/hauler_controllers.yaml</parameters>
       <ros>
-        <namespace>hauler</namespace>
+        <namespace>$(arg ns)</namespace>
       </ros>
     </plugin>

File: src/lunar_descriptions/urdf/scout.urdf.xacro (robot description, xacro)
@@ -1,4 +1,6 @@
 <?xml version="1.0"?>
-<robot xmlns:xacro="http://www.ros.org/wiki/xacro" name="scout">
+<robot xmlns:xacro="http://www.ros.org/wiki/xacro" name="$(arg name)">
+  <xacro:arg name="name" default="scout"/>
+  <xacro:arg name="ns" default="scout"/>
   <xacro:include filename="$(find lunar_descriptions)/urdf/common.xacro"/>
   <!-- ===== 腿宏：髋 + 膝 + 足，均绕 y 轴（矢状面运动）===== -->
@@ -79,9 +81,9 @@
     <mu2>0.5</mu2>
   </gazebo>
-  <!-- ===== 四条腿 ===== -->
-  <xacro:leg prefix="fl" x="0.12" y="0.08"/>
-  <xacro:leg prefix="fr" x="0.12" y="-0.08"/>
-  <xacro:leg prefix="rl" x="-0.12" y="0.08"/>
-  <xacro:leg prefix="rr" x="-0.12" y="-0.08"/>
+  <!-- ===== 四条腿（进一步加宽横向间距，抑制侧向翻倒）===== -->
+  <xacro:leg prefix="fl" x="0.12" y="0.18"/>
+  <xacro:leg prefix="fr" x="0.12" y="-0.18"/>
+  <xacro:leg prefix="rl" x="-0.12" y="0.18"/>
+  <xacro:leg prefix="rr" x="-0.12" y="-0.18"/>
   <!-- ===== 3D 激光雷达（顶部前侧，输出 sensor_msgs/PointCloud2） ===== -->
   <link name="lidar_link">
@@ -129,9 +131,9 @@
       <plugin name="scout_lidar_3d" filename="libgazebo_ros_ray_sensor.so">
         <ros>
-          <namespace>/scout</namespace>
+          <namespace>/$(arg ns)</namespace>
           <remapping>~/out:=scan_3d</remapping>
         </ros>
         <output_type>sensor_msgs/PointCloud2</output_type>
-        <frame_name>scout/lidar_link</frame_name>
+        <frame_name>$(arg ns)/lidar_link</frame_name>
       </plugin>
     </sensor>
@@ -141,8 +143,8 @@
     <plugin filename="libgazebo_ros2_control.so" name="gazebo_ros2_control">
       <robot_param>robot_description</robot_param>
-      <robot_param_node>scout_rsp</robot_param_node>
+      <robot_param_node>$(arg name)_rsp</robot_param_node>
       <parameters>$(find lunar_control)/config/scout_controllers.yaml</parameters>
       <ros>
-        <namespace>scout</namespace>
+        <namespace>$(arg ns)</namespace>
       </ros>
     </plugin>
